File: KiCad/OTO_NO_ITA/OTO_NO_ITA.kicad_pcb (KiCad board)
At the start: 6 copper layers, 73 x 72 mm, 131 parts, among them J1 Conn_02x06_Odd_Even, J2 Conn_02x10_Odd_Even, J3 Conn_02x13_Odd_Even, J4 15910060, J5 Conn_02x07_Odd_Even, J6 Conn_02x04_Odd_Even, J7 Conn_01x02, J8 Conn_01x02, J9 UB1611-HGN, Q1 STD2805T4, Q2 STL40DN3LLH5, Q3 STL40DN3LLH5, SW1 SKRPABE010, SW2 SKRPABE010, SW3 SKRPABE010, SW4 SKRPABE010, U1 MX25UW25645GXDI00, U2 STM32H7S3Z8Tx, U3 ADAU1466WBCPZ300RL, U4 ADM811TARTZ, U5 AP7361EA-33E-13, U6 AP2127N-1.8TRG1, U7 TCPP03-M20, U8 ESDA25P35-1U1M, U9 ECMF2-40A100N6, X1 24MHz, X2 12.288MHz

Commit message: 外形寸法を記入
Other:
- board text added: "UNIT: mm PITCH: 2.54 HOLE: 3.2mm x4"
