File: KiCad/OTO_NO_TE/OTO_NO_TE.kicad_pcb (KiCad board)
At the start: 4 copper layers, 114.3 x 85 mm, 61 parts, among them J1 Conn_01x13, U1 74HC4051, U2 DRV5055A3xDBZxQ1, U3 DRV5055A3xDBZxQ1, U4 DRV5055A3xDBZxQ1, U5 DRV5055A3xDBZxQ1, U6 DRV5055A3xDBZxQ1, U7 DRV5055A3xDBZxQ1

Commit message: POT数を8から12に、磁気スイッチを6から10に変更
Parts:
- added C24: ~, Capacitor_SMD:C_0603_1608Metric_Pad1.08x0.95mm_HandSolder, B.Cu at (117.1, 125.8)
- added C25: 10nF, Capacitor_SMD:C_0402_1005Metric, B.Cu at (111.5, 125.4)
- added C26: ~, Capacitor_SMD:C_0603_1608Metric_Pad1.08x0.95mm_HandSolder, B.Cu at (136.1, 125.8)
- added C27: 10nF, Capacitor_SMD:C_0402_1005Metric, B.Cu at (130.6, 125.3)
- added C28: ~, Capacitor_SMD:C_0603_1608Metric_Pad1.08x0.95mm_HandSolder, B.Cu at (98.1, 144.8)
- added C29: 10nF, Capacitor_SMD:C_0402_1005Metric, B.Cu at (92.9, 144.3)
- added C30: ~, Capacitor_SMD:C_0603_1608Metric_Pad1.08x0.95mm_HandSolder, B.Cu at (155.2, 144.8)
- added C31: 10nF, Capacitor_SMD:C_0402_1005Metric, B.Cu at (149.9, 144.3)
- added J2: Conn_01x06, Connector_PinHeader_2.54mm:PinHeader_1x06_P2.54mm_Vertical, F.Cu at (74.4, 107.7)
- added J3: Conn_01x06, Connector_PinHeader_2.54mm:PinHeader_1x06_P2.54mm_Vertical, F.Cu at (70.6, 107.7)
- added R10: ~, Resistor_SMD:R_0603_1608Metric_Pad0.98x0.95mm_HandSolder, B.Cu at (156.9, 144.8)
- added R7: ~, Resistor_SMD:R_0603_1608Metric_Pad0.98x0.95mm_HandSolder, B.Cu at (118.8, 125.8)
- added R8: ~, Resistor_SMD:R_0603_1608Metric_Pad0.98x0.95mm_HandSolder, B.Cu at (137.9, 125.8)
- added R9: ~, Resistor_SMD:R_0603_1608Metric_Pad0.98x0.95mm_HandSolder, B.Cu at (99.7, 144.8)
- added REF**: GATERON_KS-33C_ONLY, My_Parts:GATERON_KS-33C_ONLY, F.Cu at (133.5, 121.5)
- added REF**: GATERON_KS-33C_ONLY, My_Parts:GATERON_KS-33C_ONLY, F.Cu at (95.3, 140.5)
- added REF**: GATERON_KS-33C_ONLY, My_Parts:GATERON_KS-33C_ONLY, F.Cu at (114.4, 121.5)
- added REF**: GATERON_KS-33C_ONLY, My_Parts:GATERON_KS-33C_ONLY, F.Cu at (152.5, 140.5)
- added RV10: 10k, My_Parts:RK09K1130A5R, F.Cu at (171.6, 82.4)
- added RV11: 10k, My_Parts:RK09K1130A5R, F.Cu at (114.4, 102.4)
- added RV12: 10k, My_Parts:RK09K1130A5R, F.Cu at (171.6, 102.4)
- added RV9: 10k, My_Parts:RK09K1130A5R, F.Cu at (114.4, 82.4)
- added U10: DRV5056A3QDBZR, Package_TO_SOT_SMD:SOT-23, B.Cu at (95.4, 144.8)
- added U11: DRV5056A3QDBZR, Package_TO_SOT_SMD:SOT-23, B.Cu at (152.5, 144.8)
- added U8: CD74HC4067M, Package_SO:SOIC-24W_7.5x15.4mm_P1.27mm, B.Cu at (86.2, 111.0)
- added U9: DRV5056A3QDBZR, Package_TO_SOT_SMD:SOT-23, B.Cu at (133.5, 125.8)
- C1: moved to B.Cu
- J1: value Conn_01x13 -> Conn_01x06; footprint Connector_PinHeader_2.54mm:PinHeader_1x13_P2.54mm_Vertical -> Connector_PinHeader_2.54mm:PinHeader_1x06_P2.54mm_Vertical; moved to F.Cu
- RV1, RV2, RV3, RV4, RV5, RV6, RV7, RV8: value R_Potentiometer -> 10k
- U1: value 74HC4051 -> DRV5056A3QDBZR; footprint Package_SO:TSSOP-16-1EP_4.4x5mm_P0.65mm -> Package_TO_SOT_SMD:SOT-23; moved to B.Cu
- U2, U3, U4, U5, U6, U7: value DRV5055A3xDBZxQ1 -> DRV5056A3QDBZR
- moved U1 50.8 mm to (114.4, 125.8), turned to -90 degrees
- moved C1 30.6 mm to (90.0, 119.7), turned to 180 degrees
- moved J1 26.9 mm to (78.2, 107.7), turned to 0 degrees
- moved RV5 19.1 mm to (95.3, 82.4)
- moved RV7 19.1 mm to (95.3, 102.4)
- moved RV1 19.0 mm to (76.3, 82.4)
- moved RV3 19.0 mm to (76.3, 102.4)
- moved C11 19.0 mm to (136.3, 144.7)
- moved C5 19.0 mm to (130.5, 144.3)
- moved R4 19.0 mm to (138.0, 144.7)
- moved U4 19.0 mm to (114.4, 144.8)
- moved U5 19.0 mm to (133.5, 144.8)
- moved C10 19.0 mm to (117.1, 144.7)
- moved C4 19.0 mm to (111.3, 144.3)
- moved R3 19.0 mm to (118.8, 144.7)
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Connections:
- J1 pad 6: /KEY5 -> Net-(J1-Pin_6)
- U1 pad 1: /R0 -> VCC
- U1 pad 2: /R2 -> /KEY6
- U1 pad 3: Net-(J1-Pin_5) -> GND
Routing:
- net /L5: track 0.00 -> 108.2 mm, vias 0 -> 1
- net /KEY9: track 0.00 -> 96.7 mm, vias 0 -> 2
- net /R5: track 0.00 -> 89.0 mm, vias 0 -> 1
- net /KEY7: track 0.00 -> 58.1 mm
- net /L4: track 0.00 -> 51.6 mm
- net /KEY8: track 0.00 -> 46.2 mm, vias 0 -> 2
- net /KEY6: track 0.00 -> 38.6 mm
- net /R4: track 0.00 -> 38.4 mm, vias 0 -> 1
- net GND: track 62.3 -> 95.2 mm, vias 22 -> 32
- net /L3: track 51.9 -> 22.3 mm, vias 1 -> 0
- net /KEY4: track 103.7 -> 124.7 mm
- net /R2: track 76.7 -> 97.2 mm, vias 0 -> 1
- net /KEY3: track 83.6 -> 100.7 mm
- net /KEY5: track 132.6 -> 149.4 mm
- net /R0: track 54.5 -> 70.7 mm, vias 0 -> 1
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Other:
- board text added: "J1"
- board text added: "J2"
- board text added: "J3"
- board text added: "S3"
- board text added: "SUB_KEY6"
- board text added: "SUB_KEY7"
- board text added: "SUB_KEY8"
- board text added: "SUB_KEY9"
