File: KiCad/OTO_NO_TE/OTO_NO_TE.kicad_sch (KiCad schematic)
At the start: 35 parts, among them J1 Conn_01x13, U1 74HC4051, U2 DRV5055A3xDBZxQ1, U3 DRV5055A3xDBZxQ1, U4 DRV5055A3xDBZxQ1, U5 DRV5055A3xDBZxQ1, U6 DRV5055A3xDBZxQ1, U7 DRV5055A3xDBZxQ1

Commit message: 部品値を修正
Parts:
- RV1, RV2, RV3, RV4, RV5, RV6, RV7, RV8: value R_Potentiometer -> 10k
- U2, U3, U4, U5, U6, U7: value DRV5055A3xDBZxQ1 -> DRV5056A3QDBZR
Changed lines of the file:
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@@
 			)
 		)
-		(property "Value" "R_Potentiometer"
+		(property "Value" "10k"
 			(at 193.04 71.12 0)
 			(effects
@@
 			)
 		)
-		(property "Value" "DRV5055A3xDBZxQ1"
+		(property "Value" "DRV5056A3QDBZR"
 			(at 95.25 124.206 90)
 			(effects
@@
 			)
 		)
-		(property "Value" "R_Potentiometer"
+		(property "Value" "10k"
 			(at 227.33 49.53 0)
 			(effects
@@
 			)
 		)
-		(property "Value" "DRV5055A3xDBZxQ1"
+		(property "Value" "DRV5056A3QDBZR"
 			(at 166.37 124.206 90)
 			(effects
@@
 			)
 		)
-		(property "Value" "DRV5055A3xDBZxQ1"
+		(property "Value" "DRV5056A3QDBZR"
 			(at 130.81 124.206 90)
 			(effects
@@
 			)
 		)
-		(property "Value" "R_Potentiometer"
+		(property "Value" "10k"
 			(at 227.33 92.71 0)
 			(effects
@@
 			)
 		)
-		(property "Value" "R_Potentiometer"
+		(property "Value" "10k"
 			(at 193.04 92.71 0)
 			(effects
@@
 			)
 		)
-		(property "Value" "DRV5055A3xDBZxQ1"
+		(property "Value" "DRV5056A3QDBZR"
 			(at 237.49 124.206 90)
 			(effects
@@
 			)
 		)
-		(property "Value" "R_Potentiometer"
+		(property "Value" "10k"
 			(at 227.33 71.12 0)
 			(effects
@@
 			)
 		)
-		(property "Value" "DRV5055A3xDBZxQ1"
+		(property "Value" "DRV5056A3QDBZR"
 			(at 201.93 124.206 90)
 			(effects
@@
 			)
 		)
-		(property "Value" "R_Potentiometer"
+		(property "Value" "10k"
 			(at 193.04 27.94 0)
 			(effects
@@
 			)
 		)
-		(property "Value" "R_Potentiometer"
+		(property "Value" "10k"
 			(at 227.33 27.94 0)
 			(effects
@@
 			)
 		)
-		(property "Value" "R_Potentiometer"
+		(property "Value" "10k"
 			(at 193.04 49.53 0)
 			(effects
@@
 			)
 		)
-		(property "Value" "DRV5055A3xDBZxQ1"
+		(property "Value" "DRV5056A3QDBZR"
 			(at 59.69 124.206 90)
 			(effects

Commit message: POT数を8から12に、磁気スイッチを6から10に変更
Parts:
- removed J1: Conn_01x13, Connector_PinHeader_2.54mm:PinHeader_1x13_P2.54mm_Vertical, symbol Connector_Generic:Conn_01x13
- removed U1: 74HC4051, Package_SO:TSSOP-16-1EP_4.4x5mm_P0.65mm, symbol 74xx:74HC4051
- added C24, C26, C28, C30: ~, Capacitor_SMD:C_0603_1608Metric_Pad1.08x0.95mm_HandSolder, symbol Device:C
- added C25, C27, C29, C31: 10nF, Capacitor_SMD:C_0402_1005Metric, symbol Device:C
- added J1, J2, J3: Conn_01x06, Connector_PinHeader_2.54mm:PinHeader_1x06_P2.54mm_Vertical, symbol Connector_Generic:Conn_01x06
- added R10, R7, R8, R9: ~, Resistor_SMD:R_0603_1608Metric_Pad0.98x0.95mm_HandSolder, symbol Device:R
- added RV10, RV11, RV12, RV9: 10k, My_Parts:RK09K1130A5R, symbol Device:R_Potentiometer
- added U1, U10, U11, U9: DRV5056A3QDBZR, Package_TO_SOT_SMD:SOT-23, symbol Sensor_Magnetic:DRV5055A3xDBZxQ1
- added U8: CD74HC4067M, Package_SO:SOIC-24W_7.5x15.4mm_P1.27mm, symbol 74xx:CD74HC4067M
Connections:
- net GND: now also C24.2, C25.2, C26.2, C27.2, C28.2, C29.2, C30.2, C31.2, J3.6 (Pin_6), RV10.1, RV11.1, RV12.1, RV9.1, U1.3 (GND), U10.3 (GND), U11.3 (GND), U8.12 (GND), U8.15 (~{E}), U9.3 (GND)
- net KEY0: now also J2.1 (Pin_1)
- net KEY1: now also J2.2 (Pin_2)
- net KEY2: now also J2.3 (Pin_3)
- net KEY3: now also J2.4 (Pin_4)
- net KEY4: now also J2.5 (Pin_5)
- net KEY5: now also J2.6 (Pin_6)
- net L0: now also U8.9 (I0)
- net L1: now also U8.8 (I1)
- net L2: now also U8.7 (I2)
- net L3: now also U8.6 (I3)
- net LEDs/DIN: now also J3.5 (Pin_5)
- net R0: now also U8.3 (I6)
- net R1: now also U8.2 (I7)
- net R2: now also U8.23 (I8)
- net R3: now also U8.22 (I9)
- net VCC: now also C25.1, C27.1, C29.1, C31.1, J1.1 (Pin_1), R10.1, R7.1, R8.1, R9.1, RV10.3, RV11.3, RV12.3, RV9.3, U1.1 (VCC), U10.1 (VCC), U11.1 (VCC), U8.24 (VCC), U9.1 (VCC)
- new net: J1.6 (Pin_6), U8.1 (COM)
- new net: J1.2 (Pin_2), U8.10 (S0)
- new net: J1.3 (Pin_3), U8.11 (S1)
- new net: J1.5 (Pin_5), U8.13 (S3)
- new net: J1.4 (Pin_4), U8.14 (S2)
- new net KEY6: C24.1, R7.2, U1.2 (OUT), U8.19 (I12)
- new net KEY7: C26.1, R8.2, U8.18 (I13), U9.2 (OUT)
- new net KEY8: C28.1, R9.2, U10.2 (OUT), U8.17 (I14)
- new net KEY9: C30.1, R10.2, U11.2 (OUT), U8.16 (I15)
- new net L4: RV9.2, U8.5 (I4)
- new net L5: RV10.2, U8.4 (I5)
- new net R4: RV11.2, U8.21 (I10)
- new net R5: RV12.2, U8.20 (I11)
- no-connect marks 0 -> 4
Other:
- moved on the sheet: C1, C10, C11, C12, C13, C2, C3, C4, C5, C6, C7, C8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
